Commit message: urdf

File: my_robot/urdf/robot.urdf (robot description, URDF)
Before this commit: robot lidar_robot, 4 links, 3 joints
Links:
- link base_laser: geometry visual cylinder length=0.014 radius=0.0175
- link base_link: geometry visual box size=0.24 0.16 0.04
Joints:
- joint base_joint: origin xyz=0 0 0.05 -> xyz=0 0 0.049
- joint imu_joint: origin xyz=0 0 0.08 rpy=0 0 0 -> xyz=0.075 0 0.055 rpy=0 0 1.5708
- joint laser_joint: origin xyz=0.08 0 0.14 rpy=0 0 0 -> xyz=0.10 0 0.133 rpy=0 0 0

Commit message: measurements

File: my_robot/urdf/robot.urdf (robot description, URDF)
Before this commit: robot lidar_robot, 4 links, 3 joints
Links:
- added link left_front_wheel; visual cylinder length=0.03 radius=0.049
- added link left_rear_wheel; visual cylinder length=0.03 radius=0.049
- added link right_front_wheel; visual cylinder length=0.03 radius=0.049
- added link right_rear_wheel; visual cylinder length=0.03 radius=0.049
Joints:
- added joint left_front_wheel_joint: type fixed, parent base_link, child left_front_wheel, origin xyz=0.11 0.0825 0
- added joint left_rear_wheel_joint: type fixed, parent base_link, child left_rear_wheel, origin xyz=-0.11 0.0825 0
- added joint right_front_wheel_joint: type fixed, parent base_link, child right_front_wheel, origin xyz=0.11 -0.0825 0
- added joint right_rear_wheel_joint: type fixed, parent base_link, child right_rear_wheel, origin xyz=-0.11 -0.0825 0
